File: deliverables/lighting/hardware/led/lighting_led.sch (EAGLE design)
At the start: 17 parts, among them J1 5055780671, J2 5055780671

Commit message: Added Supporting Files for V0.2
SCH, BRD, and PNG for both
Also FBX models
Parts:
- J1, J2: value 5055780671 -> MOLEX-MICROLOCK-6PIN; device Molex Micro-Lock PLUS 6-pin (90deg):5055780671 -> Molex Micro-Lock PLUS 6-Pin 90deg:MOLEX-MICROLOCK-6PIN
- LED1, LED2, LED3: value XLAMP_XP-G3_ROYAL -> XP-G3_BLUE; device XLAMP XP-G3 Royal Blue:XLAMP_XP-G3_ROYAL -> XLAMP XP-G3:XP-G3_BLUE
- LED10, LED11, LED12: value XLAMP_XP-G3_PHOTO -> XP-G3_RED; device XLAMP XP-G3 Photo Red:XLAMP_XP-G3_PHOTO -> XLAMP XP-G3:XP-G3_RED
- LED13, LED14, LED15: device XLAMP XP-E2 Far Red:XLAMP_XP-E2 -> Cree XLAMP XP-E2:XLAMP_XP-E2
- LED4, LED5, LED6: value XLAMP_XP-G3_COOL -> XP-G3_COOL; device XLAMP XP-G3 Cool White:XLAMP_XP-G3_COOL -> XLAMP XP-G3:XP-G3_COOL
- LED7, LED8, LED9: value XLAMP_XP-G3_WARM -> XP-G3_WARM; device XLAMP XP-G3 Warm White:XLAMP_XP-G3_WARM -> XLAMP XP-G3:XP-G3_WARM
