File: subsystems/automation/hardware/schematics/automation.brd (EAGLE design)
At the start: 107 x 57 mm, 2 parts, among them U1 RASPBERRY PI ZERO 2 W, U2 ESP32FEATHERV2ESP32FEATHERV2H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

Commit message: Automation Gerber, Readme
Parts:
- U1: device Raspberry Pi Zero W:RASPBERRYPI_BASTELSTUBE_V13_RASPI_BOARD_B+_FULL -> Raspberry Pi Zero 2 W:RASPBERRYPI_BASTELSTUBE_V13_RASPI_BOARD_B+_FULL
- U2: value ESP32FEATHERV2ESP32FEATHERV2HEADERS -> Adafruit ESP32 Feather V2
Changed lines of the file:
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@@
 </drillsymbolsettings>
 </settings>
-<grid distance="100" unitdist="mil" unit="mil" style="lines" multiple="1" display="yes" altdistance="5" altunitdist="mil" altunit="mil"/>
+<grid distance="100" unitdist="mil" unit="mil" style="lines" multiple="1" display="no" altdistance="5" altunitdist="mil" altunit="mil"/>
 <layers>
 <layer number="1" name="Top" color="4" fill="1" visible="yes" active="yes"/>
@@
 <layer number="33" name="tFinish" color="6" fill="3" visible="no" active="yes"/>
 <layer number="34" name="bFinish" color="6" fill="6" visible="no" active="yes"/>
-<layer number="35" name="tGlue" color="7" fill="4" visible="no" active="yes"/>
+<layer number="35" name="tGlue" color="7" fill="4" visible="yes" active="yes"/>
 <layer number="36" name="bGlue" color="7" fill="5" visible="no" active="yes"/>
 <layer number="37" name="tTest" color="7" fill="1" visible="no" active="yes"/>
@@
 </autorouter>
 <elements>
-<element name="U1" library="Raspberry Pi Zero W" library_urn="urn:adsk.wipprod:fs.file:vf.0Niv2XteR2OEI_HsVnvPwQ" package="RASPBERRYPI_BASTELSTUBE_V13_RASPI_BOARD_B+_FULL" value="RASPBERRY PI ZERO 2 W" x="5" y="-2.5" smashed="yes">
+<element name="U1" library="Raspberry Pi Zero 2 W" library_urn="urn:adsk.wipprod:fs.file:vf.0Niv2XteR2OEI_HsVnvPwQ" package="RASPBERRYPI_BASTELSTUBE_V13_RASPI_BOARD_B+_FULL" value="RASPBERRY PI ZERO 2 W" x="5" y="-2.5" smashed="yes">
 <attribute name="NAME" x="12.62" y="27.98" size="1.27" layer="25"/>
 </element>
-<element name="U2" library="ESP32 Feather V2 Socket" library_urn="urn:adsk.wipprod:fs.file:vf.wOf9326mQT6ImOG0pQpvSw" package="ESP32FEATHERV2HEADERS" value="ESP32FEATHERV2ESP32FEATHERV2HEADERS" x="93.98" y="43.18" smashed="yes" rot="R90">
+<element name="U2" library="ESP32 Feather V2 Socket" library_urn="urn:adsk.wipprod:fs.file:vf.wOf9326mQT6ImOG0pQpvSw" package="ESP32FEATHERV2HEADERS" value="Adafruit ESP32 Feather V2" base_value="Adafruit ESP32 Feather V2" x="93.98" y="43.18" smashed="yes" rot="R90">
 <attribute name="CATEGORY_L1" value="" x="93.98" y="43.18" size="1.778" layer="27" rot="R90" display="off"/>
 <attribute name="CATEGORY_L2" value="" x="93.98" y="43.18" size="1.778" layer="27" rot="R90" display="off"/>
@@
 <attribute name="MANUFACTURER" value="" x="93.98" y="43.18" size="1.778" layer="27" rot="R90" display="off"/>
 <attribute name="MPN" value="" x="93.98" y="43.18" size="1.778" layer="27" rot="R90" display="off"/>
+<attribute name="NAME" x="72.136" y="-1.27" size="1.27" layer="25" rot="R90"/>
 <attribute name="PACKAGE" value="" x="93.98" y="43.18" size="1.778" layer="27" rot="R90" display="off"/>
 <attribute name="VENDOR" value="" x="93.98" y="43.18" size="1.778" layer="27" rot="R90" display="off"/>
