File: subsystems/automation/hardware/schematics/automation.sch (EAGLE design)
At the start: 2 parts, among them U1 RASPBERRY PI ZERO 2 W, U2 ESP32FEATHERV2ESP32FEATHERV2H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

Commit message: Automation Gerber, Readme
Parts:
- U1: device Raspberry Pi Zero W:RPI-ZERO -> Raspberry Pi Zero 2 W:RPI-ZERO
- U2: value ESP32FEATHERV2ESP32FEATHERV2HEADERS -> Adafruit ESP32 Feather V2
Changed lines of the file:
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@@
 </classes>
 <parts>
-<part name="U1" library="Raspberry Pi Zero W" library_urn="urn:adsk.wipprod:fs.file:vf.0Niv2XteR2OEI_HsVnvPwQ" deviceset="RPI-ZERO" device="" value="RASPBERRY PI ZERO 2 W"/>
-<part name="U2" library="ESP32 Feather V2 Socket" library_urn="urn:adsk.wipprod:fs.file:vf.wOf9326mQT6ImOG0pQpvSw" deviceset="ESP32FEATHERV2" device="ESP32FEATHERV2HEADERS"/>
+<part name="U1" library="Raspberry Pi Zero 2 W" library_urn="urn:adsk.wipprod:fs.file:vf.0Niv2XteR2OEI_HsVnvPwQ" deviceset="RPI-ZERO" device="" value="RASPBERRY PI ZERO 2 W"/>
+<part name="U2" library="ESP32 Feather V2 Socket" library_urn="urn:adsk.wipprod:fs.file:vf.wOf9326mQT6ImOG0pQpvSw" deviceset="ESP32FEATHERV2" device="ESP32FEATHERV2HEADERS" value="Adafruit ESP32 Feather V2"/>
 </parts>
 <sheets>
@@
 <attribute name="VALUE" x="-17.78" y="-37.465" size="1.27" layer="96" font="vector"/>
 </instance>
-<instance part="U2" gate="G$1" x="-10.16" y="-5.08" smashed="yes"/>
+<instance part="U2" gate="G$1" x="-10.16" y="-5.08" smashed="yes">
+<attribute name="NAME" x="-2.54" y="18.542" size="1.778" layer="95"/>
+<attribute name="VALUE" x="-2.54" y="16.002" size="1.778" layer="96"/>
+</instance>
 </instances>
 <busses>
@@
 <segment>
 <wire x1="27.94" y1="-45.72" x2="30.48" y2="-45.72" width="0.1524" layer="91"/>
+<label x="30.48" y="-45.72" size="1.778" layer="95" xref="yes"/>
 <pinref part="U1" gate="G$1" pin="GND@8"/>
-<label x="30.48" y="-45.72" size="1.778" layer="95" xref="yes"/>
 </segment>
 <segment>
-<pinref part="U2" gate="G$1" pin="GND"/>
 <wire x1="-7.62" y1="5.08" x2="-10.16" y2="5.08" width="0.1524" layer="91"/>
 <label x="-10.16" y="5.08" size="1.778" layer="95" rot="R180" xref="yes"/>
+<pinref part="U2" gate="G$1" pin="GND"/>
 </segment>
 </net>
@@
 <segment>
 <wire x1="27.94" y1="-48.26" x2="30.48" y2="-48.26" width="0.1524" layer="91"/>
+<label x="30.48" y="-48.26" size="1.778" layer="95" xref="yes"/>
 <pinref part="U1" gate="G$1" pin="TXD0/GPIO14"/>
-<label x="30.48" y="-48.26" size="1.778" layer="95" xref="yes"/>
 </segment>
 <segment>
-<pinref part="U2" gate="G$1" pin="RX"/>
 <wire x1="-7.62" y1="-20.32" x2="-10.16" y2="-20.32" width="0.1524" layer="91"/>
 <label x="-10.16" y="-20.32" size="1.778" layer="95" rot="R180" xref="yes"/>
+<pinref part="U2" gate="G$1" pin="RX"/>
 </segment>
 </net>
@@
 <segment>
 <wire x1="27.94" y1="-50.8" x2="30.48" y2="-50.8" width="0.1524" layer="91"/>
+<label x="30.48" y="-50.8" size="1.778" layer="95" xref="yes"/>
 <pinref part="U1" gate="G$1" pin="RXD0/GPIO15"/>
-<label x="30.48" y="-50.8" size="1.778" layer="95" xref="yes"/>
 </segment>
 <segment>
-<pinref part="U2" gate="G$1" pin="TX"/>
 <wire x1="-7.62" y1="-22.86" x2="-10.16" y2="-22.86" width="0.1524" layer="91"/>
 <label x="-10.16" y="-22.86" size="1.778" layer="95" rot="R180" xref="yes"/>
+<pinref part="U2" gate="G$1" pin="TX"/>
 </segment>
 </net>
 <net name="MOSI" class="0">
 <segment>
-<pinref part="U1" gate="G$1" pin="GPIO12"/>
 <wire x1="27.94" y1="-78.74" x2="30.48" y2="-78.74" width="0.1524" layer="91"/>
 <label x="30.48" y="-78.74" size="1.778" layer="95" xref="yes"/>
+<pinref part="U1" gate="G$1" pin="GPIO12"/>
 </segment>
 <segment>
-<pinref part="U2" gate="G$1" pin="MOSI"/>
 <wire x1="-7.62" y1="-15.24" x2="-10.16" y2="-15.24" width="0.1524" layer="91"/>
 <label x="-10.16" y="-15.24" size="1.778" layer="95" rot="R180" xref="yes"/>
+<pinref part="U2" gate="G$1" pin="MOSI"/>
 </segment>
 </net>
 <net name="MISO" class="0">
 <segment>
-<pinref part="U1" gate="G$1" pin="GPIO13"/>
 <wire x1="-20.32" y1="-81.28" x2="-22.86" y2="-81.28" width="0.1524" layer="91"/>
 <label x="-22.86" y="-81.28" size="1.778" layer="95" rot="R180" xref="yes"/>
+<pinref part="U1" gate="G$1" pin="GPIO13"/>
 </segment>
 <segment>
-<pinref part="U2" gate="G$1" pin="MISO"/>
 <wire x1="-7.62" y1="-17.78" x2="-10.16" y2="-17.78" width="0.1524" layer="91"/>
 <label x="-10.16" y="-17.78" size="1.778" layer="95" rot="R180" xref="yes"/>
+<pinref part="U2" gate="G$1" pin="MISO"/>
 </segment>
 </net>
 <net name="RST" class="0">
 <segment>
-<pinref part="U1" gate="G$1" pin="GPIO5"/>
 <wire x1="-20.32" y1="-76.2" x2="-22.86" y2="-76.2" width="0.1524" layer="91"/>
 <label x="-22.86" y="-76.2" size="1.778" layer="95" rot="R180" xref="yes"/>
+<pinref part="U1" gate="G$1" pin="GPIO5"/>
 </segment>
 </net>
 <net name="SCK" class="0">
 <segment>
-<pinref part="U1" gate="G$1" pin="GPIO6"/>
 <wire x1="-20.32" y1="-78.74" x2="-22.86" y2="-78.74" width="0.1524" layer="91"/>
 <label x="-22.86" y="-78.74" size="1.778" layer="95" rot="R180" xref="yes"/>
+<pinref part="U1" gate="G$1" pin="GPIO6"/>
 </segment>
 <segment>
-<pinref part="U2" gate="G$1" pin="SCK"/>
 <wire x1="-7.62" y1="-12.7" x2="-10.16" y2="-12.7" width="0.1524" layer="91"/>
 <label x="-10.16" y="-12.7" size="1.778" layer="95" rot="R180" xref="yes"/>
+<pinref part="U2" gate="G$1" pin="SCK"/>
 </segment>
 </net>
 <net name="+5V" class="0">
 <segment>
-<pinref part="U1" gate="G$1" pin="5V0@2"/>
 <wire x1="27.94" y1="-43.18" x2="27.94" y2="-40.64" width="0.1524" layer="91"/>
 <wire x1="27.94" y1="-40.64" x2="30.48" y2="-40.64" width="0.1524" layer="91"/>
-<pinref part="U1" gate="G$1" pin="5V0@1"/>
 <junction x="27.94" y="-40.64"/>
 <label x="30.48" y="-40.64" size="1.778" layer="95" xref="yes"/>
+<pinref part="U1" gate="G$1" pin="5V0@1"/>
+<pinref part="U1" gate="G$1" pin="5V0@2"/>
 </segment>
 <segment>
-<pinref part="U2" gate="G$1" pin="+5V"/>
 <wire x1="17.78" y1="-2.54" x2="20.32" y2="-2.54" width="0.1524" layer="91"/>
 <label x="20.32" y="-2.54" size="1.778" layer="95" xref="yes"/>
+<pinref part="U2" gate="G$1" pin="+5V"/>
 </segment>
 </net>
